File: driverDisplayLED/driverDisplayLED.sch (KiCad schematic (older format))
At the start: 45 parts, among them J1 Conn_01x12_Male, J2 Conn_01x12_Male, J3 Conn_01x12_Male, J4 Conn_02x08_Counter_Clockwise, J5 Conn_01x12_Male, J6 Conn_01x12_Male, J7 Conn_01x12_Male, J8 Conn_01x12_Male, J9 Conn_01x12_Male, U1 74HC245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

Commit message: Conecto las matrices LED
Parts:
- removed C4, C7, C8, C9: C, Capacitor_SMD:CP_Elec_3x5.3, symbol Device:C
- removed J2, J3, J5, J6, J7, J8, J9: Conn_01x12_Male, Connector_PinHeader_1.00mm:PinHeader_1x12_P1.00mm_Vertical, symbol Connector:Conn_01x12_Male
- removed L1, L2, L? (x2): LedMatrix_M, symbol myLedMatrix:LedMatrix_M
- removed unit 4 of U6
- removed unit 5 of U6
- removed unit 6 of U6
- added C? (x8): C, Capacitor_SMD:CP_Elec_3x5.3, symbol Device:C
- added J? (x15): Conn_01x12_Male, Connector_PinHeader_1.00mm:PinHeader_1x12_P1.00mm_Vertical, symbol Connector:Conn_01x12_Male
- added J?: Conn_02x08_Counter_Clockwise, Connector_PinHeader_2.54mm:PinHeader_2x08_P2.54mm_Vertical, symbol Connector_Generic:Conn_02x08_Counter_Clockwise
- added L? (x8): LedMatrix_M, symbol myLedMatrix:LedMatrix_M
- added Q? (x8): FDS4953, SOIC127P600X175-8N, symbol driverDisplayLED-rescue:FDS4953-FDS4953
- added RN? (x3): R_Network04, Resistor_THT:R_Array_SIP4, symbol Device:R_Network04
- added U? (x4): 74HC595, Package_SO:HTSSOP-16-1EP_4.4x5mm_P0.65mm_EP3.4x5mm, symbol 74xx:74HC595
- added U?: 74HC138D, Package_SO:TSSOP-16_4.4x5mm_P0.65mm, symbol driverDisplayLED-rescue:74HC138D-74HC138D
Connections:
- net labels added: E1, E3, H1, H2, H3, H4, LT, SRCLK-2
- net labels removed: B4-E3, B5-E2, bus.R8-R1
- wire segments 393 -> 724
- no-connect marks 7 -> 5
Other:
- moved on the sheet: C1, C2, C3, C5, C6, D1, D2, J1, J4, Q?A, Q?B, R1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
