File: driverDisplayLED/driverDisplayLED.kicad_pcb (KiCad board)
At the start: 2 copper layers, 36 parts, among them J1 Conn_01x12_Male, J2 Conn_01x12_Male, J3 Conn_01x12_Male, J4 Conn_02x08_Row_Letter_First, J5 Conn_01x12_Male, J6 Conn_01x12_Male, J7 Conn_01x12_Male, J8 Conn_01x12_Male, J9 Conn_01x12_Male, Q1 FDS4953-FDS4953, Q2 FDS4953-FDS4953, Q3 FDS4953-FDS4953, Q4 FDS4953-FDS4953, U1 74HC245, U2 74HC595, U3 74HC595, U4 74HC245, U5 74HC138D, U6 74HC04, U7 74HC595, U8 74HC595

Commit message: cambio conector 2x08 J4
Parts:
- J4: value Conn_02x08_Row_Letter_First -> Conn_02x08_Counter_Clockwise; footprint Connector_IDC:IDC-Header_2x08_P2.54mm_Vertical -> Connector_PinHeader_2.54mm:PinHeader_2x08_P2.54mm_Vertical
- moved U1 139.6 mm to (35.1, 171.2)
- moved U5 103.1 mm to (107.8, 172.3)
- moved U4 97.4 mm to (86.2, 170.6)
- moved J4 96.7 mm to (58.3, 160.4)
- moved Q2 95.9 mm to (150.0, 171.2)
- moved RN1 73.7 mm to (179.5, 117.7)
- moved Q4 49.9 mm to (170.2, 136.4)
- moved U3 47.0 mm to (161.3, 122.5), turned to 270 degrees
- moved J2 44.8 mm to (110.8, 91.6)
- moved Q3 37.3 mm to (117.2, 142.1)
- moved U7 35.1 mm to (108.2, 123.6), turned to 270 degrees
- moved U6 32.7 mm to (131.2, 112.5), turned to 180 degrees
- moved Q1 32.2 mm to (130.8, 138.2)
- moved U2 29.3 mm to (125.7, 123.0), turned to 270 degrees
- moved U8 28.1 mm to (143.4, 122.7), turned to 270 degrees
Connections:
- J4 pad 1: (no net) -> GND
- J4 pad 10: (no net) -> /B4-b7
- J4 pad 11: (no net) -> /B2-b6
- J4 pad 12: (no net) -> /B0-b5
- J4 pad 13: (no net) -> Net-(J4-Pad13)
- J4 pad 14: (no net) -> Net-(J4-Pad14)
- J4 pad 15: (no net) -> Net-(J4-Pad15)
- J4 pad 16: (no net) -> Net-(J4-Pad16)
- J4 pad 2: (no net) -> GND
- J4 pad 3: (no net) -> GND
- J4 pad 4: (no net) -> /a4-A5
- J4 pad 5: (no net) -> /B1-a5
- J4 pad 6: (no net) -> /B3-a6
- J4 pad 7: (no net) -> Net-(J4-Pad7)
- J4 pad 8: (no net) -> GND
- J4 pad 9: (no net) -> /B5B6B7-b8
- U4 pad 3: Net-(J4-Padb1) -> Net-(J4-Pad16)
- U4 pad 4: Net-(J4-Padb2) -> Net-(J4-Pad15)
- U4 pad 5: Net-(J4-Padb3) -> Net-(J4-Pad14)
- U4 pad 6: Net-(J4-Padb4) -> Net-(J4-Pad13)

Commit message: agrego borde PCB de muestra, y sus cotas
Other:
- board outline added: 230.3 x 110.5 mm
Changed lines of the file:
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@@
   (general
     (thickness 1.6)
-    (drawings 0)
+    (drawings 6)
     (tracks 0)
     (zones 0)
@@
     )
   )
+  (dimension 230.290115 (width 0.15) (layer Dwgs.User)
+    (gr_text "230,290 mm" (at 145.108446 26.604694 359.9427764) (layer Dwgs.User)
+      (effects (font (size 1 1) (thickness 0.15)))
+    )
+    (feature1 (pts (xy 260.25 30.17) (xy 260.252733 27.433273)))
+    (feature2 (pts (xy 29.96 29.94) (xy 29.962733 27.203273)))
+    (crossbar (pts (xy 29.962148 27.789693) (xy 260.252148 28.019693)))
+    (arrow1a (pts (xy 260.252148 28.019693) (xy 259.125059 28.604988)))
+    (arrow1b (pts (xy 260.252148 28.019693) (xy 259.12623 27.432147)))
+    (arrow2a (pts (xy 29.962148 27.789693) (xy 31.088066 28.377239)))
+    (arrow2b (pts (xy 29.962148 27.789693) (xy 31.089237 27.204398)))
+  )
+  (dimension 109.920022 (width 0.15) (layer Dwgs.User)
+    (gr_text "109,920 mm" (at 263.344999 85.118045 270.0364875) (layer Dwgs.User)
+      (effects (font (size 1 1) (thickness 0.15)))
+    )
+    (feature1 (pts (xy 260.31 140.08) (xy 262.666419 140.078499)))
+    (feature2 (pts (xy 260.24 30.16) (xy 262.596419 30.158499)))
+    (crossbar (pts (xy 262.009999 30.158873) (xy 262.079999 140.078873)))
+    (arrow1a (pts (xy 262.079999 140.078873) (xy 261.492861 138.952743)))
+    (arrow1b (pts (xy 262.079999 140.078873) (xy 262.665702 138.951996)))
+    (arrow2a (pts (xy 262.009999 30.158873) (xy 261.424296 31.28575)))
+    (arrow2b (pts (xy 262.009999 30.158873) (xy 262.597137 31.285003)))
+  )
+  (gr_line (start 30.43 140.04) (end 29.99 30.09) (layer Edge.Cuts) (width 0.05))
+  (gr_line (start 260.28 139.88) (end 30.43 140.04) (layer Edge.Cuts) (width 0.05))
+  (gr_line (start 260.3 30.11) (end 260.28 140.28) (layer Edge.Cuts) (width 0.05))
+  (gr_line (start 30.14 29.82) (end 260.3 30.11) (layer Edge.Cuts) (width 0.05))
 )

Commit message: agrego modulo myLedMatrix. Probar instanciar debido al path local
Parts:
- moved C1 475.0 mm to (598.1, 278.6)
- moved C2 475.0 mm to (594.7, 285.0)
- moved C3 475.0 mm to (601.5, 288.3)
- moved C5 475.0 mm to (592.9, 297.3)
- moved C7 475.0 mm to (601.5, 283.4)
- moved C8 475.0 mm to (592.9, 292.4)
- moved D1 475.0 mm to (540.9, 306.3)
- moved J4 475.0 mm to (490.5, 357.4)
- moved J6 475.0 mm to (557.1, 288.6)
- moved J7 475.0 mm to (553.7, 288.6)
- moved J8 475.0 mm to (570.5, 288.6)
- moved R3 475.0 mm to (604.6, 270.3)
- moved U2 475.0 mm to (557.9, 320.0)
- moved U3 475.0 mm to (593.6, 319.4)
- moved U4 475.0 mm to (518.4, 367.6)
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Other:
- board size 230.3 x 110.5 mm -> 906 x 496.6 mm

Commit message: place components into PCB
Parts:
- added C10: C, Capacitor_SMD:CP_Elec_3x5.3, F.Cu at (157.4, 187.5)
- added C11: C, Capacitor_SMD:CP_Elec_3x5.3, F.Cu at (157.4, 182.6)
- added C12: C, Capacitor_SMD:CP_Elec_3x5.3, F.Cu at (157.4, 177.8)
- added C13: C, Capacitor_SMD:CP_Elec_3x5.3, F.Cu at (140.3, 196.1)
- added J10: Conn_01x12_Male, Connector_PinHeader_1.00mm:PinHeader_1x12_P1.00mm_Vertical, F.Cu at (98.0, 20.0)
- added J11: Conn_01x12_Male, Connector_PinHeader_1.00mm:PinHeader_1x12_P1.00mm_Vertical, F.Cu at (98.0, 24.0)
- added J12: Conn_01x12_Male, Connector_PinHeader_1.00mm:PinHeader_1x12_P1.00mm_Vertical, F.Cu at (98.0, 32.0)
- added J13: Conn_01x12_Male, Connector_PinHeader_1.00mm:PinHeader_1x12_P1.00mm_Vertical, F.Cu at (98.0, 37.0)
- added J14: Conn_01x12_Male, Connector_PinHeader_1.00mm:PinHeader_1x12_P1.00mm_Vertical, F.Cu at (116.0, 20.0)
- added J15: Conn_01x12_Male, Connector_PinHeader_1.00mm:PinHeader_1x12_P1.00mm_Vertical, F.Cu at (116.0, 24.0)
- added J16: Conn_01x12_Male, Connector_PinHeader_1.00mm:PinHeader_1x12_P1.00mm_Vertical, F.Cu at (116.0, 32.0)
- added J17: Conn_01x12_Male, Connector_PinHeader_1.00mm:PinHeader_1x12_P1.00mm_Vertical, F.Cu at (116.0, 37.0)
- added J18: Conn_02x08_Counter_Clockwise, Connector_PinHeader_2.54mm:PinHeader_2x08_P2.54mm_Vertical, F.Cu at (337.5, 105.0)
- added Q5: FDS4953, FDS4953:SOIC127P600X175-8N, F.Cu at (160.6, 117.5)
- added Q6: FDS4953, FDS4953:SOIC127P600X175-8N, F.Cu at (275.0, 117.5)
- added Q7: FDS4953, FDS4953:SOIC127P600X175-8N, F.Cu at (167.5, 117.5)
- added Q8: FDS4953, FDS4953:SOIC127P600X175-8N, F.Cu at (282.5, 117.5)
- added RN2: R_Network04, Resistor_THT:R_Array_SIP4, F.Cu at (108.9, 196.6)
- added RN3: R_Network04, Resistor_THT:R_Array_SIP4, F.Cu at (129.5, 178.2)
- added RN4: R_Network04, Resistor_THT:R_Array_SIP4, F.Cu at (134.9, 144.2)
- added RN5: R_Network04, Resistor_THT:R_Array_SIP4, F.Cu at (108.9, 192.3)
- added U10: 74HC595, Package_SO:HTSSOP-16-1EP_4.4x5mm_P0.65mm_EP3.4x5mm, F.Cu at (220.0, 75.0)
- added U11: 74HC595, Package_SO:HTSSOP-16-1EP_4.4x5mm_P0.65mm_EP3.4x5mm, F.Cu at (260.0, 75.0)
- added U12: 74HC595, Package_SO:HTSSOP-16-1EP_4.4x5mm_P0.65mm_EP3.4x5mm, F.Cu at (295.0, 75.0)
- added U13: 74HC595, Package_SO:HTSSOP-16-1EP_4.4x5mm_P0.65mm_EP3.4x5mm, F.Cu at (335.0, 75.0)
- added U9: 74HC138D, Package_SO:TSSOP-16_4.4x5mm_P0.65mm, F.Cu at (190.0, 115.0)
- Q1, Q2, Q3, Q4: value FDS4953-FDS4953 -> FDS4953
- moved J1 568.5 mm to (66.0, 20.0), turned to 270 degrees
- moved J3 560.0 mm to (66.0, 32.0), turned to 270 degrees
- moved J5 554.7 mm to (66.0, 37.0), turned to 270 degrees
- moved J8 551.7 mm to (82.0, 32.0), turned to 270 degrees
- moved U2 546.0 mm to (70.0, 75.0), turned to 90 degrees
- moved J6 545.7 mm to (82.0, 20.0), turned to 270 degrees
- moved J2 545.6 mm to (66.0, 24.0), turned to 270 degrees
- moved U3 541.9 mm to (110.0, 75.0), turned to 90 degrees
- moved J7 540.8 mm to (82.0, 24.0), turned to 270 degrees
- moved J9 531.6 mm to (82.0, 37.0), turned to 270 degrees
- moved U6 495.1 mm to (127.5, 75.0), turned to 90 degrees
- moved U5 489.8 mm to (120.0, 117.5)
- moved U4 486.6 mm to (102.5, 115.0)
- moved Q1 484.7 mm to (130.0, 117.5), turned to 90 degrees
- moved J4 484.1 mm to (77.5, 105.0)
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Connections:
- net /B4-E3 renamed Net-(U4-Pad14)
- net /B5-E2 renamed Net-(U4-Pad13)
- net Net-(U1-Pad6) renamed LT
- net Net-(U1-Pad9) renamed SRCLK-2
- J1 pad 1: GND -> /R8
- J1 pad 10: /R6 -> /H3
- J1 pad 11: /R7 -> /H2
- J1 pad 12: /R8 -> /H1
- J1 pad 2: GND -> /R7
- J1 pad 3: GND -> /R6
- J1 pad 4: GND -> /R5
- J1 pad 5: /R1 -> /R4
- J1 pad 6: /R2 -> /R3
- J1 pad 7: /R3 -> /R2
- J1 pad 8: /R4 -> /R1
- J1 pad 9: /R5 -> /H4
- J2 pad 1: /H8 -> /G8
- J2 pad 10: /G6 -> /H6
- J2 pad 11: /G7 -> /H7
- J2 pad 12: /G8 -> /H8
- J2 pad 2: /H7 -> /G7
- J2 pad 3: /H6 -> /G6
- J2 pad 4: /H5 -> /G5
- J2 pad 5: /G1 -> /G4
- J2 pad 6: /G2 -> /G3
- J2 pad 7: /G3 -> /G2
- J2 pad 8: /G4 -> /G1
- J2 pad 9: /G5 -> /H5
- J3 pad 1: /H8 -> /R8
- J3 pad 10: /G6 -> /H3
- J3 pad 11: /G7 -> /H2
- J3 pad 12: /G8 -> /H1
- J3 pad 2: /H7 -> /R7
- J3 pad 3: /H6 -> /R6
- J3 pad 4: /H5 -> /R5
- J3 pad 5: /G1 -> /R4
- J3 pad 6: /G2 -> /R3
- J3 pad 7: /G3 -> /R2
- J3 pad 8: /G4 -> /R1
- J3 pad 9: /G5 -> /H4
- J5 pad 1: GND -> /G8
- J5 pad 10: /R6 -> /H6
- J5 pad 11: /R7 -> /H7
- J5 pad 12: /R8 -> /H8
- J5 pad 2: GND -> /G7
- J5 pad 3: GND -> /G6
- J5 pad 4: GND -> /G5
- J5 pad 5: /R1 -> /G4
- J5 pad 6: /R2 -> /G3
- J5 pad 7: /R3 -> /G2
- J5 pad 8: /R4 -> /G1
- J5 pad 9: /R5 -> /H5
- J6 pad 1: /H8 -> /R8
- J6 pad 10: /G6 -> /H3
- J6 pad 11: /G7 -> /H2
- J6 pad 12: /G8 -> /H1
- J6 pad 2: /H7 -> /R7
- J6 pad 3: /H6 -> /R6
- J6 pad 4: /H5 -> /R5
- J6 pad 5: /G1 -> /R4
- J6 pad 6: /G2 -> /R3
- J6 pad 7: /G3 -> /R2
- J6 pad 8: /G4 -> /R1
- J6 pad 9: /G5 -> /H4
- J7 pad 1: /H8 -> /G8
- J7 pad 10: /G6 -> /H6
- J7 pad 11: /G7 -> /H7
- J7 pad 12: /G8 -> /H8
- J7 pad 2: /H7 -> /G7
- J7 pad 3: /H6 -> /G6
- J7 pad 4: /H5 -> /G5
- J7 pad 5: /G1 -> /G4
- J7 pad 6: /G2 -> /G3
- J7 pad 7: /G3 -> /G2
- J7 pad 8: /G4 -> /G1
- J7 pad 9: /G5 -> /H5
- J8 pad 1: GND -> /R8
- J8 pad 10: /R6 -> /H3
- J8 pad 11: /R7 -> /H2
- J8 pad 12: /R8 -> /H1
- J8 pad 2: GND -> /R7
- J8 pad 3: GND -> /R6
- J8 pad 4: GND -> /R5
- J8 pad 5: /R1 -> /R4
- J8 pad 6: /R2 -> /R3
- J8 pad 7: /R3 -> /R2
- J8 pad 8: /R4 -> /R1
- J8 pad 9: /R5 -> /H4
- J9 pad 1: GND -> /G8
- J9 pad 10: /R6 -> /H6
- J9 pad 11: /R7 -> /H7
- J9 pad 12: /R8 -> /H8
- J9 pad 2: GND -> /G7
- J9 pad 3: GND -> /G6
- J9 pad 4: GND -> /G5
- J9 pad 5: /R1 -> /G4
- J9 pad 6: /R2 -> /G3
- J9 pad 7: /R3 -> /G2
- J9 pad 8: /R4 -> /G1
- J9 pad 9: /R5 -> /H5
- Q1 pad 1: /1 -> VCC
- Q1 pad 2: /2 -> /Y1-G1
- Q1 pad 3: /3 -> VCC
- Q1 pad 4: /4 -> /Y0-G2
- Q1 pad 5: /5 -> /D2-H1
- Q1 pad 6: /5 -> /D2-H1
- Q1 pad 7: /7 -> /D1-H2
- Q1 pad 8: /7 -> /D1-H2
- Q2 pad 1: /1 -> VCC
- Q2 pad 2: /2 -> /Y1-G1
- Q2 pad 3: /3 -> VCC
- Q2 pad 4: /4 -> /Y0-G2
- Q2 pad 5: /5 -> /D2-H1
- Q2 pad 6: /5 -> /D2-H1
- Q2 pad 7: /7 -> /D1-H2
- Q2 pad 8: /7 -> /D1-H2
- Q3 pad 1: /1 -> VCC
- Q3 pad 2: /2 -> /Y3-G1
- Q3 pad 3: /3 -> VCC
- Q3 pad 4: /4 -> /Y2-G2
- Q3 pad 5: /5 -> /D2-H3
- Q3 pad 6: /5 -> /D2-H3
- Q3 pad 7: /7 -> /D1-H4
- Q3 pad 8: /7 -> /D1-H4
- Q4 pad 1: /1 -> VCC
- Q4 pad 2: /2 -> /Y3-G1
- Q4 pad 3: /3 -> VCC
- Q4 pad 4: /4 -> /Y2-G2
- Q4 pad 5: /5 -> /D2-H3
- Q4 pad 6: /5 -> /D2-H3
- Q4 pad 7: /7 -> /D1-H4
- Q4 pad 8: /7 -> /D1-H4
- R2 pad 1: Net-(R2-Pad1) -> Net-(C6-Pad1)
- RN1 pad 1: Net-(RN1-Pad1) -> GND
- RN1 pad 2: Net-(RN1-Pad2) -> /D2-H1
- RN1 pad 3: Net-(RN1-Pad3) -> /D1-H2
- RN1 pad 4: Net-(RN1-Pad4) -> /D2-H3
- U1 pad 1: Net-(U1-Pad1) -> GND
- U1 pad 19: Net-(U1-Pad19) -> GND
- U2 pad 1: Net-(U2-Pad1) -> /R7
- U2 pad 15: Net-(U2-Pad15) -> /R8
- U2 pad 2: Net-(U2-Pad2) -> /R6
- U2 pad 3: Net-(U2-Pad3) -> /R5
- U2 pad 4: Net-(U2-Pad4) -> /R4
- U2 pad 5: Net-(U2-Pad5) -> /R3
- U2 pad 6: Net-(U2-Pad6) -> /R2
- U2 pad 7: Net-(U2-Pad7) -> /R1
- U3 pad 9: /QH-SER -> Net-(U3-Pad9)
- U5 pad 12: /4 -> Net-(U5-Pad12)
- U5 pad 13: /2 -> Net-(U5-Pad13)
- U5 pad 14: /4 -> Net-(U5-Pad14)
- U5 pad 15: /2 -> Net-(U5-Pad15)
- U5 pad 4: Net-(U5-Pad4) -> /E1
- U6 pad 1: Net-(R2-Pad1) -> Net-(C6-Pad1)
- U6 pad 10: Net-(U6-Pad10) -> (no net)
- U6 pad 11: VCC -> (no net)
- U6 pad 12: Net-(U6-Pad12) -> (no net)
- U6 pad 13: VCC -> (no net)
- U6 pad 4: Net-(U6-Pad4) -> /E1
- U6 pad 5: Net-(U6-Pad4) -> /E1
- U6 pad 6: Net-(U6-Pad6) -> /E3
- U6 pad 8: Net-(U6-Pad8) -> (no net)
- U6 pad 9: VCC -> (no net)
- U7 pad 14: /A1-SER -> Net-(U3-Pad9)
- U7 pad 9: /QH-SER -> Net-(U7-Pad9)
- U8 pad 14: /A1-SER -> Net-(U7-Pad9)
Other:
- board outline removed

Commit message: place components, continued
Parts:
- J1, J10, J11, J12, J13, J14, J15, J16, J17, J2, J3, J5, J6, J7, J8, J9: footprint Connector_PinHeader_1.00mm:PinHeader_1x12_P1.00mm_Vertical -> Connector_PinSocket_2.54mm:PinSocket_1x12_P2.54mm_Vertical
- U1, U4: footprint Package_SO:HSOP-20-1EP_11.0x15.9mm_P1.27mm_SlugDown_ThermalVias -> Package_SO:SO-20-1EP_7.52x12.825mm_P1.27mm_EP6.045x12.09mm_Mask3.56x4.47mm
- U10, U11, U12, U13, U2, U3, U7, U8: footprint Package_SO:HTSSOP-16-1EP_4.4x5mm_P0.65mm_EP3.4x5mm -> Package_SO:SO-16_5.3x10.2mm_P1.27mm
- U5, U9: footprint Package_SO:TSSOP-16_4.4x5mm_P0.65mm -> Package_SO:SO-16_5.3x10.2mm_P1.27mm
- moved C2 220.9 mm to (60.0, 75.0), turned to 90 degrees
- moved C5 173.2 mm to (122.5, 70.0), turned to 270 degrees
- moved R3 165.2 mm to (120.0, 85.0)
- moved C10 164.5 mm to (307.4, 120.0)
- moved C11 164.5 mm to (307.4, 115.1)
- moved C12 164.5 mm to (307.4, 110.3)
- moved C9 164.5 mm to (314.2, 110.3)
- moved C13 164.5 mm to (290.3, 128.6)
- moved C6 156.5 mm to (126.5, 85.0)
- moved R1 139.0 mm to (115.0, 85.0)
- moved D2 136.4 mm to (116.8, 79.7), turned to 90 degrees
- moved D1 135.8 mm to (120.0, 80.0), turned to 270 degrees
- moved R2 135.5 mm to (117.5, 85.0)
- moved C4 129.0 mm to (102.5, 75.0), turned to 90 degrees
- moved J17 126.7 mm to (202.6, 129.5)
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
Commit message: agrego textos. Listo para revisión esquemático
Parts:
- removed C10, C12, C13, C9: C, Capacitor_SMD:CP_Elec_3x5.3
- removed RN1, RN3, RN4, RN5: R_Network04, Resistor_THT:R_Array_SIP4
- removed U10, U11, U12, U13: 74HC595, Package_SO:SO-16_5.3x10.2mm_P1.27mm
- added RN6: 50, Resistor_THT:R_Array_SIP4, F.Cu at (168.2, 42.7)
- added RN7: 50, Resistor_THT:R_Array_SIP4, F.Cu at (180.3, 42.7)
- added RN8: 50, Resistor_THT:R_Array_SIP4, F.Cu at (192.4, 42.7)
- added RN9: 50, Resistor_THT:R_Array_SIP4, F.Cu at (204.5, 42.7)
- moved J5 145.6 mm to (172.9, 10.3), turned to 0 degrees
- moved J9 135.4 mm to (191.3, 10.3), turned to 0 degrees
- moved J13 127.1 mm to (209.7, 10.3), turned to 0 degrees
- moved J17 121.9 mm to (228.1, 10.3), turned to 0 degrees
- moved J3 119.1 mm to (168.3, 10.3), turned to 0 degrees
- moved J8 106.8 mm to (186.7, 10.3), turned to 0 degrees
- moved J7 98.4 mm to (182.1, 10.3), turned to 0 degrees
- moved J12 97.1 mm to (205.1, 10.3), turned to 0 degrees
- moved J16 91.0 mm to (223.5, 10.3), turned to 0 degrees
- moved J11 89.3 mm to (200.5, 10.3), turned to 0 degrees
- moved J15 84.2 mm to (218.9, 10.3), turned to 0 degrees
- moved J6 71.9 mm to (177.5, 10.3), turned to 0 degrees
- moved J10 60.4 mm to (195.9, 10.3), turned to 0 degrees
- moved J14 53.4 mm to (214.3, 10.3), turned to 0 degrees
Connections:
- J1 pad 1: /R8 -> /L1R8
- J1 pad 10: /H3 -> /H3a
- J1 pad 11: /H2 -> /H2a
- J1 pad 12: /H1 -> /H1a
- J1 pad 2: /R7 -> /L1R7
- J1 pad 3: /R6 -> /L1R6
- J1 pad 4: /R5 -> /L1R5
- J1 pad 5: /R4 -> /L1R4
- J1 pad 6: /R3 -> /L1R3
- J1 pad 7: /R2 -> /L1R2
- J1 pad 8: /R1 -> /L1R1
- J1 pad 9: /H4 -> /H4a
- J10 pad 1: /R8 -> /L5R8
- J10 pad 10: /H3 -> /H3a
- J10 pad 11: /H2 -> /H2a
- J10 pad 12: /H1 -> /H1a
- J10 pad 2: /R7 -> /L5R7
- J10 pad 3: /R6 -> /L5R6
- J10 pad 4: /R5 -> /L5R5
- J10 pad 5: /R4 -> /L5R4
- J10 pad 6: /R3 -> /L5R3
- J10 pad 7: /R2 -> /L5R2
- J10 pad 8: /R1 -> /L5R1
- J10 pad 9: /H4 -> /H4a
- J11 pad 1: /G8 -> Net-(J11-Pad1)
- J11 pad 10: /H6 -> /H6a
- J11 pad 11: /H7 -> /H7a
- J11 pad 12: /H8 -> /H8a
- J11 pad 2: /G7 -> Net-(J11-Pad2)
- J11 pad 3: /G6 -> Net-(J11-Pad3)
- J11 pad 4: /G5 -> Net-(J11-Pad4)
- J11 pad 5: /G4 -> Net-(J11-Pad5)
- J11 pad 6: /G3 -> Net-(J11-Pad6)
- J11 pad 7: /G2 -> Net-(J11-Pad7)
- J11 pad 8: /G1 -> Net-(J11-Pad8)
- J11 pad 9: /H5 -> /H5a
- J12 pad 1: /R8 -> /L5R8
- J12 pad 10: /H3 -> /H3b
- J12 pad 11: /H2 -> /H2b
- J12 pad 12: /H1 -> /H1b
- J12 pad 2: /R7 -> /L5R7
- J12 pad 3: /R6 -> /L5R6
- J12 pad 4: /R5 -> /L5R5
- J12 pad 5: /R4 -> /L5R4
- J12 pad 6: /R3 -> /L5R3
- J12 pad 7: /R2 -> /L5R2
- J12 pad 8: /R1 -> /L5R1
- J12 pad 9: /H4 -> /H4b
- J13 pad 1: /G8 -> GND
- J13 pad 10: /H6 -> /H6b
- J13 pad 11: /H7 -> /H7b
- J13 pad 12: /H8 -> /H8b
- J13 pad 2: /G7 -> GND
- J13 pad 3: /G6 -> GND
- J13 pad 4: /G5 -> GND
- J13 pad 5: /G4 -> GND
- J13 pad 6: /G3 -> GND
- J13 pad 7: /G2 -> GND
- J13 pad 8: /G1 -> GND
- J13 pad 9: /H5 -> /H5b
- J14 pad 1: /R8 -> /L7R8
- J14 pad 10: /H3 -> /H3a
- J14 pad 11: /H2 -> /H2a
- J14 pad 12: /H1 -> /H1a
- J14 pad 2: /R7 -> /L7R7
- J14 pad 3: /R6 -> /L7R6
- J14 pad 4: /R5 -> /L7R5
- J14 pad 5: /R4 -> /L7R4
- J14 pad 6: /R3 -> /L7R3
- J14 pad 7: /R2 -> /L7R2
- J14 pad 8: /R1 -> /L7R1
- J14 pad 9: /H4 -> /H4a
- J15 pad 1: /G8 -> /L7G8
- J15 pad 10: /H6 -> /H6a
- J15 pad 11: /H7 -> /H7a
- J15 pad 12: /H8 -> /H8a
- J15 pad 2: /G7 -> /L7G7
- J15 pad 3: /G6 -> /L7G6
- J15 pad 4: /G5 -> /L7G5
- J15 pad 5: /G4 -> /L7G4
- J15 pad 6: /G3 -> /L7G3
- J15 pad 7: /G2 -> /L7G2
- J15 pad 8: /G1 -> /L7G1
- J15 pad 9: /H5 -> /H5a
- J16 pad 1: /R8 -> /L7R8
- J16 pad 10: /H3 -> /H3b
- J16 pad 11: /H2 -> /H2b
- J16 pad 12: /H1 -> /H1b
- J16 pad 2: /R7 -> /L7R7
- J16 pad 3: /R6 -> /L7R6
- J16 pad 4: /R5 -> /L7R5
- J16 pad 5: /R4 -> /L7R4
- J16 pad 6: /R3 -> /L7R3
- J16 pad 7: /R2 -> /L7R2
- J16 pad 8: /R1 -> /L7R1
- J16 pad 9: /H4 -> /H4b
- J17 pad 1: /G8 -> GND
- J17 pad 10: /H6 -> /H6b
- J17 pad 11: /H7 -> /H7b
- J17 pad 12: /H8 -> /H8b
- J17 pad 2: /G7 -> GND
- J17 pad 3: /G6 -> GND
- J17 pad 4: /G5 -> GND
- J17 pad 5: /G4 -> GND
- J17 pad 6: /G3 -> GND
- J17 pad 7: /G2 -> GND
- J17 pad 8: /G1 -> GND
- J17 pad 9: /H5 -> /H5b
- J2 pad 1: /G8 -> /L1G8
- J2 pad 10: /H6 -> /H6a
- J2 pad 11: /H7 -> /H7a
- J2 pad 12: /H8 -> /H8a
- J2 pad 2: /G7 -> /L1G7
- J2 pad 3: /G6 -> /L1G6
- J2 pad 4: /G5 -> /L1G5
- J2 pad 5: /G4 -> /L1G4
- J2 pad 6: /G3 -> /L1G3
- J2 pad 7: /G2 -> /L1G2
- J2 pad 8: /G1 -> /L1G1
- J2 pad 9: /H5 -> /H5a
- J3 pad 1: /R8 -> /L1R8
- J3 pad 10: /H3 -> /H3b
- J3 pad 11: /H2 -> /H2b
- J3 pad 12: /H1 -> /H1b
- J3 pad 2: /R7 -> /L1R7
- J3 pad 3: /R6 -> /L1R6
- J3 pad 4: /R5 -> /L1R5
- J3 pad 5: /R4 -> /L1R4
- J3 pad 6: /R3 -> /L1R3
- J3 pad 7: /R2 -> /L1R2
- J3 pad 8: /R1 -> /L1R1
- J3 pad 9: /H4 -> /H4b
- J5 pad 1: /G8 -> GND
- J5 pad 10: /H6 -> /H6b
- J5 pad 11: /H7 -> /H7b
- J5 pad 12: /H8 -> /H8b
- J5 pad 2: /G7 -> GND
- J5 pad 3: /G6 -> GND
- J5 pad 4: /G5 -> GND
- J5 pad 5: /G4 -> GND
- J5 pad 6: /G3 -> GND
- J5 pad 7: /G2 -> GND
- J5 pad 8: /G1 -> GND
- J5 pad 9: /H5 -> /H5b
- J6 pad 1: /R8 -> /L3R8
- J6 pad 10: /H3 -> /H3a
- J6 pad 11: /H2 -> /H2a
- J6 pad 12: /H1 -> /H1a
- J6 pad 2: /R7 -> /L3R7
- J6 pad 3: /R6 -> /L3R6
- J6 pad 4: /R5 -> /L3R5
- J6 pad 5: /R4 -> /L3R4
- J6 pad 6: /R3 -> /L3R3
- J6 pad 7: /R2 -> /L3R2
- J6 pad 8: /R1 -> /L3R1
- J6 pad 9: /H4 -> /H4a
- J7 pad 1: /G8 -> Net-(J7-Pad1)
- J7 pad 10: /H6 -> /H6a
- J7 pad 11: /H7 -> /H7a
- J7 pad 12: /H8 -> /H8a
- J7 pad 2: /G7 -> Net-(J7-Pad2)
- J7 pad 3: /G6 -> Net-(J7-Pad3)
- J7 pad 4: /G5 -> Net-(J7-Pad4)
- J7 pad 5: /G4 -> Net-(J7-Pad5)
- J7 pad 6: /G3 -> Net-(J7-Pad6)
- J7 pad 7: /G2 -> Net-(J7-Pad7)
- J7 pad 8: /G1 -> Net-(J7-Pad8)
- J7 pad 9: /H5 -> /H5a
- J8 pad 1: /R8 -> /L3R8
- J8 pad 10: /H3 -> /H3b
- J8 pad 11: /H2 -> /H2b
- J8 pad 12: /H1 -> /H1b
- J8 pad 2: /R7 -> /L3R7
- J8 pad 3: /R6 -> /L3R6
- J8 pad 4: /R5 -> /L3R5
- J8 pad 5: /R4 -> /L3R4
- J8 pad 6: /R3 -> /L3R3
- J8 pad 7: /R2 -> /L3R2
- J8 pad 8: /R1 -> /L3R1
- J8 pad 9: /H4 -> /H4b
- J9 pad 1: /G8 -> GND
- J9 pad 10: /H6 -> /H6b
- J9 pad 11: /H7 -> /H7b
- J9 pad 12: /H8 -> /H8b
- J9 pad 2: /G7 -> GND
- J9 pad 3: /G6 -> GND
- J9 pad 4: /G5 -> GND
- J9 pad 5: /G4 -> GND
- J9 pad 6: /G3 -> GND
- J9 pad 7: /G2 -> GND
- J9 pad 8: /G1 -> GND
- J9 pad 9: /H5 -> /H5b
- Q1 pad 2: /Y1-G1 -> /Y1-G1b
- Q1 pad 4: /Y0-G2 -> /Y0-G2b
- Q1 pad 5: /D2-H1 -> /H5b
- Q1 pad 6: /D2-H1 -> /H5b
- Q1 pad 7: /D1-H2 -> /H6b
- Q1 pad 8: /D1-H2 -> /H6b
- Q2 pad 2: /Y1-G1 -> /Y1-G1a
- Q2 pad 4: /Y0-G2 -> /Y0-G2a
- Q2 pad 5: /D2-H1 -> /H5a
- Q2 pad 6: /D2-H1 -> /H5a
- Q2 pad 7: /D1-H2 -> /H6a
- Q2 pad 8: /D1-H2 -> /H6a
- Q3 pad 2: /Y3-G1 -> /Y3-G1b
- Q3 pad 4: /Y2-G2 -> /Y2-G2b
- Q3 pad 5: /D2-H3 -> /H7b
- Q3 pad 6: /D2-H3 -> /H7b
- Q3 pad 7: /D1-H4 -> /H8b
- Q3 pad 8: /D1-H4 -> /H8b
- Q4 pad 2: /Y3-G1 -> /Y3-G1a
- Q4 pad 4: /Y2-G2 -> /Y2-G2a
- Q4 pad 5: /D2-H3 -> /H7a
- Q4 pad 6: /D2-H3 -> /H7a
- Q4 pad 7: /D1-H4 -> /H8a
- Q4 pad 8: /D1-H4 -> /H8a
- Q5 pad 2: /Y5-G1 -> /Y5-G1b
- Q5 pad 4: /Y4-G2 -> /Y4-G2b
- Q5 pad 5: Net-(Q5-Pad5) -> /H4b
- Q5 pad 6: Net-(Q5-Pad5) -> /H4b
- Q5 pad 7: Net-(Q5-Pad7) -> /H3b
- Q5 pad 8: Net-(Q5-Pad7) -> /H3b
- Q6 pad 2: /Y5-G1 -> /Y5-G1a
- Q6 pad 4: /Y4-G2 -> /Y4-G2a
- Q6 pad 5: Net-(Q6-Pad5) -> /H4a
- Q6 pad 6: Net-(Q6-Pad5) -> /H4a
- Q6 pad 7: Net-(Q6-Pad7) -> /H3a
- Q6 pad 8: Net-(Q6-Pad7) -> /H3a
- Q7 pad 2: /Y7-G1 -> /Y7-G1b
- Q7 pad 4: /Y6-G2 -> /Y6-G2b
- Q7 pad 5: Net-(Q7-Pad5) -> /H2b
- Q7 pad 6: Net-(Q7-Pad5) -> /H2b
- Q7 pad 7: Net-(Q7-Pad7) -> /H1b
- Q7 pad 8: Net-(Q7-Pad7) -> /H1b
- Q8 pad 2: /Y7-G1 -> /Y7-G1a
- Q8 pad 4: /Y6-G2 -> /Y6-G2a
- Q8 pad 5: Net-(Q8-Pad5) -> /H2a
- Q8 pad 6: Net-(Q8-Pad5) -> /H2a
- Q8 pad 7: Net-(Q8-Pad7) -> /H1a
- Q8 pad 8: Net-(Q8-Pad7) -> /H1a
- U2 pad 1: /R7 -> /L1R7
- U2 pad 15: /R8 -> /L1R8
- U2 pad 2: /R6 -> /L1R6
- U2 pad 3: /R5 -> /L1R5
- U2 pad 4: /R4 -> /L1R4
- U2 pad 5: /R3 -> /L1R3
- U2 pad 6: /R2 -> /L1R2
- U2 pad 7: /R1 -> /L1R1
- U2 pad 9: /QH-SER -> Net-(U2-Pad9)
- U3 pad 1: Net-(U3-Pad1) -> /L3R7
- U3 pad 14: /QH-SER -> Net-(U2-Pad9)
- U3 pad 15: Net-(U3-Pad15) -> /L3R8
- U3 pad 2: Net-(U3-Pad2) -> /L3R6
- U3 pad 3: Net-(U3-Pad3) -> /L3R5
- U3 pad 4: Net-(U3-Pad4) -> /L3R4
- U3 pad 5: Net-(U3-Pad5) -> /L3R3
- U3 pad 6: Net-(U3-Pad6) -> /L3R2
- U3 pad 7: Net-(U3-Pad7) -> /L3R1
- U5 pad 10: Net-(U5-Pad10) -> /Y5-G1b
- U5 pad 11: Net-(U5-Pad11) -> /Y4-G2b
- U5 pad 12: Net-(U5-Pad12) -> /Y3-G1b
- U5 pad 13: Net-(U5-Pad13) -> /Y2-G2b
- U5 pad 14: Net-(U5-Pad14) -> /Y1-G1b
- U5 pad 15: Net-(U5-Pad15) -> /Y0-G2b
- U5 pad 7: Net-(U5-Pad7) -> /Y7-G1b
- U5 pad 9: Net-(U5-Pad9) -> /Y6-G2b
- U7 pad 1: Net-(U7-Pad1) -> /L5R7
- U7 pad 15: Net-(U7-Pad15) -> /L5R8
- U7 pad 2: Net-(U7-Pad2) -> /L5R6
- U7 pad 3: Net-(U7-Pad3) -> /L5R5
- U7 pad 4: Net-(U7-Pad4) -> /L5R4
- U7 pad 5: Net-(U7-Pad5) -> /L5R3
- U7 pad 6: Net-(U7-Pad6) -> /L5R2
- U7 pad 7: Net-(U7-Pad7) -> /L5R1
- U8 pad 1: Net-(U8-Pad1) -> /L7R7
- U8 pad 15: Net-(U8-Pad15) -> /L7R8
- U8 pad 2: Net-(U8-Pad2) -> /L7R6
- U8 pad 3: Net-(U8-Pad3) -> /L7R5
- U8 pad 4: Net-(U8-Pad4) -> /L7R4
- U8 pad 5: Net-(U8-Pad5) -> /L7R3
- U8 pad 6: Net-(U8-Pad6) -> /L7R2
- U8 pad 7: Net-(U8-Pad7) -> /L7R1
- U9 pad 10: Net-(U9-Pad10) -> /Y5-G1a
- U9 pad 11: Net-(U9-Pad11) -> /Y4-G2a
- U9 pad 12: Net-(U9-Pad12) -> /Y3-G1a
- U9 pad 13: Net-(U9-Pad13) -> /Y2-G2a
- U9 pad 14: Net-(U9-Pad14) -> /Y1-G1a
- U9 pad 15: Net-(U9-Pad15) -> /Y0-G2a
- U9 pad 7: Net-(U9-Pad7) -> /Y7-G1a
- U9 pad 9: Net-(U9-Pad9) -> /Y6-G2a

Commit message: place and route
Parts:
- removed J18: Conn_02x08_Counter_Clockwise, Connector_PinHeader_2.54mm:PinHeader_2x08_P2.54mm_Vertical
- added H1: MountingHole, MountingHole:MountingHole_2.7mm_M2.5_ISO14580, F.Cu at (65.5, 67.5)
- added H2: MountingHole, MountingHole:MountingHole_2.7mm_M2.5_ISO14580, F.Cu at (66.0, 124.5)
- added H3: MountingHole, MountingHole:MountingHole_2.7mm_M2.5_ISO14580, F.Cu at (99.8, 120.8)
- added H4: MountingHole, MountingHole:MountingHole_2.7mm_M2.5_ISO14580, F.Cu at (220.1, 88.1)
- added H5: MountingHole, MountingHole:MountingHole_2.7mm_M2.5_ISO14580, F.Cu at (99.0, 72.0)
- added H6: MountingHole, MountingHole:MountingHole_2.7mm_M2.5_ISO14580, F.Cu at (226.1, 88.1)
- moved J5 162.5 mm to (63.0, 130.0), turned to 90 degrees
- moved J9 149.8 mm to (100.5, 129.5), turned to 90 degrees
- moved J13 139.2 mm to (137.8, 129.5), turned to 90 degrees
- moved J3 138.7 mm to (63.0, 100.5), turned to 90 degrees
- moved J17 130.1 mm to (175.8, 129.5), turned to 90 degrees
- moved J8 124.9 mm to (100.3, 100.5), turned to 90 degrees
- moved J7 115.9 mm to (100.3, 92.4), turned to 90 degrees
- moved J12 111.8 mm to (139.0, 100.5), turned to 90 degrees
- moved J11 102.7 mm to (138.8, 92.5), turned to 90 degrees
- moved J16 102.0 mm to (175.8, 100.5), turned to 90 degrees
- moved J6 93.9 mm to (99.5, 62.5), turned to 90 degrees
- moved J15 92.8 mm to (175.8, 92.5), turned to 90 degrees
- moved J10 78.5 mm to (137.3, 62.6), turned to 90 degrees
- moved J14 64.8 mm to (175.8, 62.5), turned to 90 degrees
- moved RN6 45.1 mm to (160.7, 87.2)
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Connections:
- J4 pad 10: /B4-b7 -> /B0-b5
- J4 pad 11: /B2-b6 -> /B3-a6
- J4 pad 12: /B0-b5 -> /B2-b6
- J4 pad 14: Net-(J4-Pad14) -> /B4-b7
- J4 pad 15: Net-(J4-Pad15) -> GND
- J4 pad 16: Net-(J4-Pad16) -> /B5B6B7-b8
- J4 pad 2: GND -> Net-(J4-Pad2)
- J4 pad 4: /a4-A5 -> Net-(J4-Pad4)
- J4 pad 5: /B1-a5 -> GND
- J4 pad 6: /B3-a6 -> Net-(J4-Pad6)
- J4 pad 7: Net-(J4-Pad7) -> /a4-A5
- J4 pad 8: GND -> Net-(J4-Pad8)
- J4 pad 9: /B5B6B7-b8 -> /B1-a5
- U4 pad 3: Net-(J4-Pad16) -> Net-(J4-Pad2)
- U4 pad 4: Net-(J4-Pad15) -> Net-(J4-Pad4)
- U4 pad 5: Net-(J4-Pad14) -> Net-(J4-Pad6)
- U4 pad 6: Net-(J4-Pad13) -> Net-(J4-Pad8)
Routing:
- net /A1-SER: track 0.00 -> 52.2 mm
- net /RCLK: track 0.00 -> 48.2 mm
- net Net-(U2-Pad9): track 0.00 -> 34.7 mm
- net /B0-b5: track 0.00 -> 15.6 mm
- net /B5B6B7-b8: track 0.00 -> 15.5 mm
- net /B4-b7: track 0.00 -> 15.2 mm
- net /B2-b6: track 0.00 -> 15.0 mm
- net /B1-a5: track 0.00 -> 10.2 mm
- net /B3-a6: track 0.00 -> 10.2 mm
- net (no net): vias 0 -> 8
- added copper zone on F.Cu, net GND
