File: driverDisplayLED/Inverters.sch (KiCad schematic (older format))
At the start: 9 parts, among them U9 74HC04

Commit message: Agrego codigos de catalogo, documentación, y linkeo del borrador del PCB
Parts:
- C8: value C -> 2u
- C9: value C -> 1u
- D1, D2: value D -> 1n4008
- R1, R2, R3: value R -> 220
- U9: CodigoCatalogo (none) -> 296-14505-2-ND - Tape & Reel (TR)
Changed lines of the file:
@@
 AR Path="/6352902C/63544E5D" Ref="C9"  Part="1"
 F 0 "C9" V 9273 3025 50  0000 C CNN
-F 1 "C" V 9364 3025 50  0000 C CNN
+F 1 "1u" V 9364 3025 50  0000 C CNN
 F 2 "Capacitor_SMD:C_0201_0603Metric" H 9563 2875 50  0001 C CNN
 F 3 "~" H 9525 3025 50  0001 C CNN
@@
 AR Path="/6352902C/63544E67" Ref="C8"  Part="1"
 F 0 "C8" V 5623 2925 50  0000 C CNN
-F 1 "C" V 5714 2925 50  0000 C CNN
+F 1 "2u" V 5714 2925 50  0000 C CNN
 F 2 "Capacitor_SMD:C_0201_0603Metric" H 5913 2775 50  0001 C CNN
 F 3 "~" H 5875 2925 50  0001 C CNN
@@
 AR Path="/6352902C/63544E82" Ref="R3"  Part="1"
 F 0 "R3" V 5525 2925 50  0000 C CNN
-F 1 "R" V 5425 2925 50  0000 C CNN
+F 1 "220" V 5425 2925 50  0000 C CNN
 F 2 "Resistor_SMD:R_0201_0603Metric" V 5255 2925 50  0001 C CNN
 F 3 "~" H 5325 2925 50  0001 C CNN
@@
 AR Path="/6352902C/63544E9B" Ref="D1"  Part="1"
 F 0 "D1" V 4704 2955 50  0000 L CNN
-F 1 "D" V 4795 2955 50  0000 L CNN
+F 1 "1n4008" V 4795 2955 50  0000 L CNN
 F 2 "Diode_SMD:D_0201_0603Metric" H 4750 2875 50  0001 C CNN
 F 3 "~" H 4750 2875 50  0001 C CNN
@@
 AR Path="/6352902C/63544EA1" Ref="D2"  Part="1"
 F 0 "D2" V 4954 2680 50  0000 L CNN
-F 1 "D" V 5045 2680 50  0000 L CNN
+F 1 "1n4008" V 5045 2680 50  0000 L CNN
 F 2 "Diode_SMD:D_0201_0603Metric" H 5000 2600 50  0001 C CNN
 F 3 "~" H 5000 2600 50  0001 C CNN
@@
 AR Path="/6352902C/63544EAE" Ref="R2"  Part="1"
 F 0 "R2" V 3700 2875 50  0000 C CNN
-F 1 "R" V 3600 2875 50  0000 C CNN
+F 1 "220" V 3600 2875 50  0000 C CNN
 F 2 "Resistor_SMD:R_0201_0603Metric" V 3430 2875 50  0001 C CNN
 F 3 "~" H 3500 2875 50  0001 C CNN
@@
 F 2 "Package_SO:SO-14_5.3x10.2mm_P1.27mm" H 9875 3075 50  0001 C CNN
 F 3 "https://assets.nexperia.com/documents/data-sheet/74HC_HCT04.pdf" H 9875 3075 50  0001 C CNN
+F 4 "296-14505-2-ND - Tape & Reel (TR)" H 9875 3075 50  0001 C CNN "CodigoCatalogo"
 	7    9875 3075
 	1    0    0    -1
@@
 AR Path="/6352902C/63544EB4" Ref="R1"  Part="1"
 F 0 "R1" V 3450 2600 50  0000 C CNN
-F 1 "R" V 3350 2600 50  0000 C CNN
+F 1 "220" V 3350 2600 50  0000 C CNN
 F 2 "Resistor_SMD:R_0201_0603Metric" V 3180 2600 50  0001 C CNN
 F 3 "~" H 3250 2600 50  0001 C CNN
