File: driverDisplayLED/arrayMOSFET.sch (KiCad schematic (older format))
At the start: 8 parts, among them Q1 FDS4953, Q2 FDS4953, Q3 FDS4953, Q4 FDS4953, Q5 FDS4953, Q6 FDS4953, Q7 FDS4953, Q8 FDS4953

Commit message: Agrego codigos de catalogo, documentación, y linkeo del borrador del PCB
Parts:
- Q1, Q2, Q3, Q4, Q5, Q6, Q7, Q8: CodigoCatalogo (none) -> FDS4953TR-ND - Tape & Reel (TR)
Changed lines of the file:
@@
 F 27 "6.0" H 6950 3825 50  0001 L BNN "Field42"
 F 28 "5.8" H 6950 3825 50  0001 L BNN "Field43"
+F 29 "FDS4953TR-ND - Tape & Reel (TR)" H 6950 3825 50  0001 C CNN "CodigoCatalogo"
 	1    6950 3825
 	1    0    0    1
@@
 F 27 "6.0" H 7550 3825 50  0001 L BNN "Field42"
 F 28 "5.8" H 7550 3825 50  0001 L BNN "Field43"
+F 29 "FDS4953TR-ND - Tape & Reel (TR)" H 7550 3825 50  0001 C CNN "CodigoCatalogo"
 	2    7550 3825
 	1    0    0    1
@@
 F 27 "6.0" H 5575 3825 50  0001 L BNN "Field42"
 F 28 "5.8" H 5575 3825 50  0001 L BNN "Field43"
+F 29 "FDS4953TR-ND - Tape & Reel (TR)" H 5575 3825 50  0001 C CNN "CodigoCatalogo"
 	1    5575 3825
 	1    0    0    1
@@
 F 27 "6.0" H 6175 3825 50  0001 L BNN "Field42"
 F 28 "5.8" H 6175 3825 50  0001 L BNN "Field43"
+F 29 "FDS4953TR-ND - Tape & Reel (TR)" H 6175 3825 50  0001 C CNN "CodigoCatalogo"
 	2    6175 3825
 	1    0    0    1
@@
 F 27 "6.0" H 5025 3825 50  0001 L BNN "Field42"
 F 28 "5.8" H 5025 3825 50  0001 L BNN "Field43"
+F 29 "FDS4953TR-ND - Tape & Reel (TR)" H 5025 3825 50  0001 C CNN "CodigoCatalogo"
 	2    5025 3825
 	1    0    0    1
@@
 F 27 "6.0" H 4425 3825 50  0001 L BNN "Field42"
 F 28 "5.8" H 4425 3825 50  0001 L BNN "Field43"
+F 29 "FDS4953TR-ND - Tape & Reel (TR)" H 4425 3825 50  0001 C CNN "CodigoCatalogo"
 	1    4425 3825
 	1    0    0    1
@@
 F 27 "6.0" H 6950 5325 50  0001 L BNN "Field42"
 F 28 "5.8" H 6950 5325 50  0001 L BNN "Field43"
+F 29 "FDS4953TR-ND - Tape & Reel (TR)" H 6950 5325 50  0001 C CNN "CodigoCatalogo"
 	1    6950 5325
 	1    0    0    1
@@
 F 27 "6.0" H 7550 5325 50  0001 L BNN "Field42"
 F 28 "5.8" H 7550 5325 50  0001 L BNN "Field43"
+F 29 "FDS4953TR-ND - Tape & Reel (TR)" H 7550 5325 50  0001 C CNN "CodigoCatalogo"
 	2    7550 5325
 	1    0    0    1
@@
 F 27 "6.0" H 8100 5325 50  0001 L BNN "Field42"
 F 28 "5.8" H 8100 5325 50  0001 L BNN "Field43"
+F 29 "FDS4953TR-ND - Tape & Reel (TR)" H 8100 5325 50  0001 C CNN "CodigoCatalogo"
 	1    8100 5325
 	1    0    0    1
@@
 F 27 "6.0" H 8700 5325 50  0001 L BNN "Field42"
 F 28 "5.8" H 8700 5325 50  0001 L BNN "Field43"
+F 29 "FDS4953TR-ND - Tape & Reel (TR)" H 8700 5325 50  0001 C CNN "CodigoCatalogo"
 	2    8700 5325
 	1    0    0    1
@@
 F 27 "6.0" H 5575 5325 50  0001 L BNN "Field42"
 F 28 "5.8" H 5575 5325 50  0001 L BNN "Field43"
+F 29 "FDS4953TR-ND - Tape & Reel (TR)" H 5575 5325 50  0001 C CNN "CodigoCatalogo"
 	1    5575 5325
 	1    0    0    1
@@
 F 27 "6.0" H 6175 5325 50  0001 L BNN "Field42"
 F 28 "5.8" H 6175 5325 50  0001 L BNN "Field43"
+F 29 "FDS4953TR-ND - Tape & Reel (TR)" H 6175 5325 50  0001 C CNN "CodigoCatalogo"
 	2    6175 5325
 	1    0    0    1
@@
 F 27 "6.0" H 5025 5325 50  0001 L BNN "Field42"
 F 28 "5.8" H 5025 5325 50  0001 L BNN "Field43"
+F 29 "FDS4953TR-ND - Tape & Reel (TR)" H 5025 5325 50  0001 C CNN "CodigoCatalogo"
 	2    5025 5325
 	1    0    0    1
@@
 F 27 "6.0" H 4425 5325 50  0001 L BNN "Field42"
 F 28 "5.8" H 4425 5325 50  0001 L BNN "Field43"
+F 29 "FDS4953TR-ND - Tape & Reel (TR)" H 4425 5325 50  0001 C CNN "CodigoCatalogo"
 	1    4425 5325
 	1    0    0    1
@@
 F 27 "6.0" H 8100 3825 50  0001 L BNN "Field42"
 F 28 "5.8" H 8100 3825 50  0001 L BNN "Field43"
+F 29 "FDS4953TR-ND - Tape & Reel (TR)" H 8100 3825 50  0001 C CNN "CodigoCatalogo"
 	1    8100 3825
 	1    0    0    1
@@
 F 27 "6.0" H 8700 3825 50  0001 L BNN "Field42"
 F 28 "5.8" H 8700 3825 50  0001 L BNN "Field43"
+F 29 "FDS4953TR-ND - Tape & Reel (TR)" H 8700 3825 50  0001 C CNN "CodigoCatalogo"
 	2    8700 3825
 	1    0    0    1
