File: driverDisplayLED/driverDisplayLED_hierarchical.sch (KiCad schematic (older format))
At the start: 7 parts, among them J19 Conn_01x02_Female

Commit message: Agrego nuevo proyecto: Modulo Infrarrojo TxRx
Changed lines of the file:
@@
 F5 "Vin" I L 2230 2790 50
 F6 "GND" I L 2230 2885 50
-F7 "L1R[1...8]" B R 4855 2710 50
-F8 "L3R[1..8]" B R 4855 2835 50
-F9 "L5R[1..8]" B R 4855 2960 50
-F10 "L7R[1..8]" B R 4855 3085 50
+F7 "L3R[1..8]" B R 4855 2835 50
+F8 "L5R[1..8]" B R 4855 2960 50
+F9 "L7R[1..8]" B R 4855 3085 50
+F10 "L1R[1..8]" B R 4855 2710 50
 $EndSheet
 Wire Wire Line
