File: driverDisplayLED/modulo_IR/modulo_IR.kicad_pcb (KiCad board)
At the start: 2 copper layers, 15 parts, among them J1 Conn_01x03_Male, U1 SFH617A-1X001, U2 LM393

Commit message: placing components
Parts:
- U1: footprint Package_SO:SO-4_7.6x3.6mm_P2.54mm -> Package_SO:SO-4_4.4x2.3mm_P1.27mm
- moved J1 34.7 mm to (157.0, 81.0)
- moved H2 30.2 mm to (117.0, 84.0)
- moved C2 27.1 mm to (122.6, 78.0)
- moved C1 27.0 mm to (122.6, 76.0)
- moved R5 24.9 mm to (123.0, 82.0)
- moved RV1 22.6 mm to (130.0, 77.0)
- moved D1 21.6 mm to (111.0, 81.5), turned to 90 degrees
- moved U1 21.3 mm to (145.0, 75.0)
- moved D2 20.1 mm to (111.0, 88.5), turned to 90 degrees
- moved R3 19.7 mm to (123.0, 84.0)
- moved R1 18.9 mm to (123.0, 80.0)
- moved R4 16.7 mm to (123.0, 86.0)
- moved H1 15.0 mm to (153.0, 83.0)
- moved U2 10.5 mm to (130.0, 86.0), turned to 90 degrees

Commit message: Diseño del PCB
Parts:
- moved R2 25.3 mm to (121.4, 83.2)
- moved H1 13.3 mm to (139.8, 84.2)
- moved R3 13.0 mm to (135.8, 86.1), turned to 90 degrees
- moved J1 9.70 mm to (147.4, 79.6)
- moved D2 8.94 mm to (111.0, 79.6)
- moved R1 7.77 mm to (121.4, 87.6)
- moved U1 6.05 mm to (139.0, 75.8), turned to 180 degrees
- moved H2 5.83 mm to (114.8, 78.6)
- moved D1 4.46 mm to (111.0, 86.0)
- moved C1 1.89 mm to (121.0, 77.0)
- moved C2 1.89 mm to (121.0, 79.0)
- moved R5 1.89 mm to (121.4, 81.0)
- moved R4 1.71 mm to (121.4, 85.4)
- moved RV1 1.02 mm to (129.8, 78.0)
- turned U2 to 0 degrees
Routing:
- net +5V: track 0.00 -> 104.4 mm
- net Net-(C2-Pad1): track 0.00 -> 41.5 mm, vias 0 -> 3
- net /D0: track 0.00 -> 29.4 mm, vias 0 -> 2
- net Net-(R3-Pad2): track 0.00 -> 13.1 mm
- net Net-(RV1-Pad2): track 0.00 -> 11.5 mm
- net Net-(D2-Pad1): track 0.00 -> 11.0 mm
- net Net-(D1-Pad1): track 0.00 -> 10.2 mm
- net (no net): track 0.00 -> 0.98 mm
- net GND: vias 0 -> 2
- added copper zone on B.Cu, net GND
- added copper zone on F.Cu, net GND
