File: driverDisplayLED/modulo_IR/_autosave-modulo_IR.sch (KiCad schematic (older format))
At the start: 16 parts, among them J1 Conn_01x03_Male, U2 LM393

Commit message: Ordeno el repo y actualizo esquemático y netlist
Parts:
- C1, C2: footprint Capacitor_SMD:C_0504_1310Metric_Pad0.83x1.28mm_HandSolder -> Capacitor_SMD:C_0805_2012Metric
- J1: footprint Connector_PinHeader_2.54mm:PinHeader_1x03_P2.54mm_Vertical -> Connector_PinHeader_2.54mm:PinHeader_1x03_P2.54mm_Horizontal
Changed lines of the file:
@@
 F 0 "C1" H 3625 2976 50  0000 L CNN
 F 1 "104" H 3625 2885 50  0000 L CNN
-F 2 "Capacitor_SMD:C_0504_1310Metric_Pad0.83x1.28mm_HandSolder" H 3548 2780 50  0001 C CNN
+F 2 "Capacitor_SMD:C_0805_2012Metric" H 3548 2780 50  0001 C CNN
 F 3 "~" H 3510 2930 50  0001 C CNN
 	1    3510 2930
@@
 F 0 "J1" H 7568 5031 50  0000 C CNN
 F 1 "Conn_01x03_Male" H 7568 4940 50  0000 C CNN
-F 2 "Connector_PinHeader_2.54mm:PinHeader_1x03_P2.54mm_Vertical" H 7460 4750 50  0001 C CNN
+F 2 "Connector_PinHeader_2.54mm:PinHeader_1x03_P2.54mm_Horizontal" H 7460 4750 50  0001 C CNN
 F 3 "~" H 7460 4750 50  0001 C CNN
 	1    7460 4750
@@
 F 0 "C2" H 6295 5716 50  0000 L CNN
 F 1 "104" H 6295 5625 50  0000 L CNN
-F 2 "Capacitor_SMD:C_0504_1310Metric_Pad0.83x1.28mm_HandSolder" H 6218 5520 50  0001 C CNN
+F 2 "Capacitor_SMD:C_0805_2012Metric" H 6218 5520 50  0001 C CNN
 F 3 "~" H 6180 5670 50  0001 C CNN
 	1    6180 5670
